Commit message: panda model modified

File: curi_sim/description/Panda/panda_bk.urdf (robot description, URDF)
Before this commit: robot panda, 12 links, 11 joints
Joints:
- joint panda_joint2: limit lower=-1.7628 upper=1.7628 effort=87 velocity=2.1750 -> lower=-1.8326 upper=1.8326 effort=87 velocity=2.1750
- joint panda_joint3: limit lower=-2.8973 upper=2.8973 effort=87 velocity=2.1750 -> lower=-2.9671 upper=2.9671 effort=87 velocity=2.1750
- joint panda_joint4: limit lower=-3.0718 upper=-0.4 effort=87 velocity=2.1750 -> lower=-3.1416 upper=0.0 effort=87 velocity=2.1750
- joint panda_joint5: limit lower=-2.8973 upper=2.8973 effort=12 velocity=2.6100 -> lower=-2.9671 upper=2.9671 effort=12 velocity=2.6100
